File: Geiger_counter_HV_section.brd (EAGLE design)
At the start: 42.1 x 26.6 mm, 22 parts, among them IC1 TLC555, Q1 MMBT3904, Q2 KSC5502

Commit message: Updated
Parts:
- R1: value 330 -> 10k
- R2: value 1k -> 330
Changed lines of the file:
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@@
 </element>
 <element name="Q2" library="thomas_library" package="TO-252" value="KSC5502" x="92.456" y="59.182" smashed="yes" rot="R270"/>
-<element name="R1" library="thomas_library" package="0805" value="330" x="84.836" y="61.468" smashed="yes" rot="R180">
+<element name="R1" library="thomas_library" package="0805" value="10k" x="84.836" y="61.468" smashed="yes" rot="R180">
 <attribute name="NAME" x="85.598" y="63.5635" size="0.6096" layer="25" rot="R180"/>
 </element>
-<element name="R2" library="thomas_library" package="0805" value="1k" x="73.152" y="63.754" smashed="yes">
+<element name="R2" library="thomas_library" package="0805" value="330" x="73.152" y="63.754" smashed="yes">
 <attribute name="NAME" x="73.66" y="65.2145" size="0.6096" layer="25"/>
 </element>
