File: Geiger_counter_uC_section.sch (EAGLE design)
At the start: 33 parts, among them IC1 ATTINY641, IC2 MCP1703, Q1 MMBT3904, Q2 MMBT3904, Q3 MMBT3904, X1 11.0592 MHz

Commit message: Updated
Parts:
- IC1: value ATTINY641 -> ATTINY841
Changed lines of the file:
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@@
 </classes>
 <parts>
-<part name="IC1" library="thomas_library" deviceset="ATTINY841" device="SO-14" package3d_urn="urn:adsk.eagle:package:16406/2" value="ATTINY641"/>
+<part name="IC1" library="thomas_library" deviceset="ATTINY841" device="SO-14" package3d_urn="urn:adsk.eagle:package:16406/2" value="ATTINY841"/>
 <part name="X1" library="thomas_library" deviceset="ABM3" device="" value="11.0592 MHz"/>
 <part name="C1" library="thomas_library" deviceset="CAPACITOR" device="0805" value="22pF"/>
